File: mpu.sch (KiCad schematic (older format))
At the start: 18 parts, among them J2 USB_B, U1 AT91SAM9N12, Y1 16MHz, Y2 32.768kHz

Commit message: Ordered boards
Parts:
- removed J2: USB_B, Connector_USB:USB_Micro-B_GCT_USB3076-30-A, symbol Connector:USB_B
- added D5: LED, LED_SMD:LED_0603_1608Metric_Pad1.05x0.95mm_HandSolder, symbol Device:LED
- added J2: USB_A, Connector_USB:USB3_A_Molex_48393-001, symbol Connector:USB_A
- added R20: 4.7k, Resistor_SMD:R_0402_1005Metric, symbol Device:R
Connections:
- net labels added: fullD+, fullD-, microD+, microD-
- wire segments 201 -> 204
Changed lines of the file:
@@
 	1    0    0    -1
 $EndComp
-Entry Wire Line
-	12100 1450 12200 1550
-Entry Wire Line
-	12100 1550 12200 1650
-Entry Wire Line
-	12100 1650 12200 1750
-Wire Wire Line
-	12200 1550 12700 1550
-Wire Wire Line
-	12200 1650 12700 1650
-Wire Wire Line
-	12200 1750 12700 1750
-Text Label 12200 1550 0    50   ~ 0
+Text Label 12150 1450 0    50   ~ 0
 actGPIO0
-Text Label 12200 1650 0    50   ~ 0
+Text Label 12150 1550 0    50   ~ 0
 actGPIO1
-Text Label 12200 1750 0    50   ~ 0
+Text Label 12150 1650 0    50   ~ 0
 actGPIO2
 Wire Bus Line
-	12700 1750 12700 1400
-Wire Bus Line
-	12700 1400 13000 1400
-Text HLabel 13000 1400 2    50   Input ~ 0
+	12650 1300 12950 1300
+Text HLabel 12950 1300 2    50   Input ~ 0
 actGPIO[0..2]
 $Comp
@@
 	1    0    0    -1
 $EndComp
-Text HLabel 12500 4700 2    50   Input ~ 0
+Text HLabel 12600 4700 2    50   Input ~ 0
 D+
-Text HLabel 12500 4800 2    50   Input ~ 0
+Text HLabel 12600 4800 2    50   Input ~ 0
 D-
 $Comp
 L Device:R R12
 U 1 1 5C0D28DC
-P 12100 4700
-F 0 "R12" V 12100 4650 50  0000 C CNN
-F 1 "22" V 12100 4750 50  0000 C CNN
-F 2 "Resistor_SMD:R_0402_1005Metric" V 12030 4700 50  0001 C CNN
-F 3 "~" H 12100 4700 50  0001 C CNN
-	1    12100 4700
+P 12200 4700
+F 0 "R12" V 12200 4650 50  0000 C CNN
+F 1 "22" V 12200 4750 50  0000 C CNN
+F 2 "Resistor_SMD:R_0402_1005Metric" V 12130 4700 50  0001 C CNN
+F 3 "~" H 12200 4700 50  0001 C CNN
+	1    12200 4700
 	0    1    1    0
 $EndComp
@@
 L Device:R R13
 U 1 1 5C0D2943
-P 12100 4800
-F 0 "R13" V 12100 4750 50  0000 C CNN
-F 1 "22" V 12100 4850 50  0000 C CNN
-F 2 "Resistor_SMD:R_0402_1005Metric" V 12030 4800 50  0001 C CNN
-F 3 "~" H 12100 4800 50  0001 C CNN
-	1    12100 4800
-	0    1    1    0
-$EndComp
-Wire Wire Line
-	11950 4700 11750 4700
-Wire Wire Line
-	12250 4700 12500 4700
-Wire Wire Line
-	12500 4800 12250 4800
-Wire Wire Line
-	11950 4800 11750 4800
-$Comp
-L Connector:USB_B J2
-U 1 1 5C109EE1
-P 11350 5700
-F 0 "J2" H 11405 6167 50  0000 C CNN
-F 1 "USB_B" H 11405 6076 50  0000 C CNN
-F 2 "Connector_USB:USB_Micro-B_GCT_USB3076-30-A" H 11500 5650 50  0001 C CNN
-F 3 " ~" H 11500 5650 50  0001 C CNN
-	1    11350 5700
-	1    0    0    -1
-$EndComp
+P 12200 4800
+F 0 "R13" V 12200 4750 50  0000 C CNN
+F 1 "22" V 12200 4850 50  0000 C CNN
+F 2 "Resistor_SMD:R_0402_1005Metric" V 12130 4800 50  0001 C CNN
+F 3 "~" H 12200 4800 50  0001 C CNN
+	1    12200 4800
+	0    1    1    0
+$EndComp
+Wire Wire Line
+	12350 4700 12600 4700
+Wire Wire Line
+	12600 4800 12350 4800
 $Comp
 L Atmel:AT91SAM9N12 U1
@@
 	1    0    0    -1
 $EndComp
+$Comp
+L Connector:USB_A J2
+U 1 1 5BCCF81D
+P 11350 5700
+F 0 "J2" H 11405 6167 50  0000 C CNN
+F 1 "USB_A" H 11405 6076 50  0000 C CNN
+F 2 "Connector_USB:USB3_A_Molex_48393-001" H 11500 5650 50  0001 C CNN
+F 3 " ~" H 11500 5650 50  0001 C CNN
+	1    11350 5700
+	1    0    0    -1
+$EndComp
+Text Label 11750 4700 0    50   ~ 0
+microD+
+Text Label 11750 4800 0    50   ~ 0
+microD-
+Wire Wire Line
+	11750 4700 12050 4700
+Wire Wire Line
+	11750 4800 12050 4800
+Text Label 11700 6850 0    50   ~ 0
+fullD+
+Text Label 11700 6950 0    50   ~ 0
+fullD-
+Entry Wire Line
+	12550 1450 12650 1550
+Entry Wire Line
+	12550 1550 12650 1650
+Wire Wire Line
+	12100 1650 12550 1650
+Wire Wire Line
+	12100 1550 12550 1550
+Wire Wire Line
+	12100 1450 12550 1450
+Entry Wire Line
+	12550 1650 12650 1750
+Wire Wire Line
+	12100 1950 12900 1950
+$Comp
+L Device:R R20
+U 1 1 5BDF477E
+P 13050 1950
+F 0 "R20" V 13050 1900 50  0000 C CNN
+F 1 "4.7k" V 13050 2050 50  0000 C CNN
+F 2 "Resistor_SMD:R_0402_1005Metric" V 12980 1950 50  0001 C CNN
+F 3 "~" H 13050 1950 50  0001 C CNN
+	1    13050 1950
+	0    1    1    0
+$EndComp
+$Comp
+L Device:LED D5
+U 1 1 5BDF4B45
+P 13350 1950
+F 0 "D5" H 13400 1850 50  0000 C CNN
+F 1 "LED" H 13100 1900 50  0000 C CNN
+F 2 "LED_SMD:LED_0603_1608Metric_Pad1.05x0.95mm_HandSolder" H 13350 1950 50  0001 C CNN
+F 3 "~" H 13350 1950 50  0001 C CNN
+	1    13350 1950
+	-1   0    0    1
+$EndComp
+$Comp
+L power:GND #PWR0165
+U 1 1 5BE63DAB
+P 13650 2050
+F 0 "#PWR0165" H 13650 1800 50  0001 C CNN
+F 1 "GND" H 13655 1877 50  0000 C CNN
+F 2 "" H 13650 2050 50  0001 C CNN
+F 3 "" H 13650 2050 50  0001 C CNN
+	1    13650 2050
+	1    0    0    -1
+$EndComp
+Wire Wire Line
+	13650 1950 13500 1950
+Wire Wire Line
+	13650 2050 13650 1950
 Wire Bus Line
 	2350 5850 2350 7450
 Wire Bus Line
+	12650 1300 12650 1750
+Wire Bus Line
 	5400 2650 5400 3350
