File: mpuBoard.sch (KiCad schematic (older format))
At the start: 0 parts

Commit message: Ordered boards
Changed lines of the file:
@@
 $EndSheet
-Wire Bus Line
-	7050 2150 7050 3800
 Wire Bus Line
 	7050 3800 6000 3800
@@
 Wire Wire Line
 	3100 3650 3700 3650
+Wire Bus Line
+	7050 2100 7050 3800
 $EndSCHEMATC
