File: nandFlash.sch (KiCad schematic (older format))
At the start: 5 parts, among them U4 S34ML08G201TFI

Commit message: Ordered boards
Changed lines of the file:
@@
 Text Notes 3250 4450 0    50   ~ 0
 flashCTL BUS DECODING\nFLASH | NET | uP\nCLE - FLASHCTL0 - NANDCLE\nALE - FLASHCTL1 - NANDALE\nWE# - FLASHCTL2 - NANDWE\nWP# - FLASHCTL3 - NC\nR/B# - FLASHCTL4 - NWAIT\nRE# - FLASHCTL5 - NANDOE\nCE# - FLASHCTL6 - NCS3\n
+$Comp
+L power:+3V3 #PWR0156
+U 1 1 5BCE69AF
+P 6200 3450
+F 0 "#PWR0156" H 6200 3300 50  0001 C CNN
+F 1 "+3V3" H 6215 3623 50  0000 C CNN
+F 2 "" H 6200 3450 50  0001 C CNN
+F 3 "" H 6200 3450 50  0001 C CNN
+	1    6200 3450
+	1    0    0    -1
+$EndComp
+Connection ~ 6200 3450
 Wire Bus Line
 	6000 3750 6000 4750
