File: power.sch (KiCad schematic (older format))
At the start: 28 parts, among them J1 USB_B_Micro, Q1 bss138, Q2 bss138, Q3 bss138, SW1 SW_Push, SW2 SW_Push, U2 ACT8865

Commit message: Ordered boards
Parts:
- added C35: 20u, Capacitor_SMD:C_0402_1005Metric, symbol Device:C_Small
- added D1, D2, D3, D4: LED, LED_SMD:LED_0603_1608Metric_Pad1.05x0.95mm_HandSolder, symbol Device:LED
- added R16, R17, R18, R19: 4.7k, Resistor_SMD:R_0402_1005Metric, symbol Device:R
- C7: value C_Small -> 100n
- SW1, SW2: footprint Button_Switch_SMD:SW_SPST_B3S-1000 -> Jumper:SolderJumper-2_P1.3mm_Open_Pad1.0x1.5mm
- U2: footprint Package_DFN_QFN:QFN-42-1EP_5x6mm_P0.4mm_EP3.7x4.7mm -> Package_DFN_QFN:QFN-32-1EP_4x4mm_P0.4mm_EP2.65x2.65mm
Connections:
- wire segments 147 -> 168
